File: Sofle_v2/PCB_TFTScreen/SofleKeyboard.kicad_pcb (KiCad board)
At the start: 2 copper layers, 287.8 x 115 mm, 113 parts, among them J1 Conn_01x13, J3 Conn_01x13, J7 Conn_01x08, J8 Conn_01x08, SW1 Rotary_Encoder_Switch, SW10 SW_PUSH, SW11 SW_PUSH, SW12 SW_PUSH, SW13 SW_PUSH, SW14 SW_PUSH, SW15 SW_PUSH, SW16 SW_PUSH, SW17 SW_PUSH, SW18 SW_PUSH, SW19 SW_PUSH, SW2 SW_PUSH, SW20 SW_PUSH, SW21 SW_PUSH, SW22 SW_PUSH, SW23 SW_PUSH, SW24 SW_PUSH, SW25 SW_PUSH, SW26 SW_PUSH, SW27 SW_PUSH, SW28 SW_PUSH, SW29 SW_PUSH, SW3 SW_PUSH, SW30 SW_PUSH, SW31 Rotary_Encoder_Switch, SW32 SW_PUSH, SW33 SW_PUSH, SW34 SW_PUSH, SW35 SW_PUSH, SW36 SW_PUSH, SW37 SW_PUSH, SW38 SW_PUSH, SW39 SW_PUSH, SW4 SW_PUSH, SW40 SW_PUSH, SW41 SW_PUSH, SW42 SW_PUSH, SW43 SW_PUSH, SW44 SW_PUSH, SW45 SW_PUSH, SW46 SW_PUSH, SW47 SW_PUSH, SW48 SW_PUSH, SW49 SW_PUSH, SW5 SW_PUSH, SW50 SW_PUSH, SW51 SW_PUSH, SW52 SW_PUSH, SW53 SW_PUSH, SW54 SW_PUSH, SW55 SW_PUSH, SW56 SW_PUSH, SW57 SW_PUSH, SW58 SW_PUSH, SW59 SW_PUSH, SW6 SW_PUSH, SW60 SW_PUSH, SW61 SW_PUSH, SW62 SW_PUSH, SW7 SW_PUSH, SW8 SW_PUSH, SW9 SW_PUSH, U1 , U10 , U11 , U12 , U13 , U14 , U15 , U16 , U17 , U18 , U19 , U2 Elite-C, U20 , U21 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

Commit message: Update file
Parts:
- added D1: D, SofleKeyboard-footprint:Diode_SOD123_2, F.Cu at (103.7, 205.7)
- added D10: D, SofleKeyboard-footprint:Diode_SOD123_2, F.Cu at (103.7, 226.1)
- added D11: D, SofleKeyboard-footprint:Diode_SOD123_2, F.Cu at (103.7, 228.6)
- added D12: D, SofleKeyboard-footprint:Diode_SOD123_2, F.Cu at (109.9, 205.7)
- added D13: D, SofleKeyboard-footprint:Diode_SOD123_2, F.Cu at (109.9, 208.2)
- added D14: D, SofleKeyboard-footprint:Diode_SOD123_2, F.Cu at (109.9, 210.8)
- added D15: D, SofleKeyboard-footprint:Diode_SOD123_2, F.Cu at (109.9, 213.3)
- added D16: D, SofleKeyboard-footprint:Diode_SOD123_2, F.Cu at (109.9, 215.8)
- added D17: D, SofleKeyboard-footprint:Diode_SOD123_2, F.Cu at (109.9, 218.4)
- added D18: D, SofleKeyboard-footprint:Diode_SOD123_2, F.Cu at (109.9, 220.9)
- added D19: D, SofleKeyboard-footprint:Diode_SOD123_2, F.Cu at (109.9, 223.5)
- added D2: D, SofleKeyboard-footprint:Diode_SOD123_2, F.Cu at (103.7, 208.2)
- added D20: D, SofleKeyboard-footprint:Diode_SOD123_2, F.Cu at (109.9, 226.1)
- added D21: D, SofleKeyboard-footprint:Diode_SOD123_2, F.Cu at (109.9, 228.6)
- added D22: D, SofleKeyboard-footprint:Diode_SOD123_2, F.Cu at (116.1, 205.7)
- added D23: D, SofleKeyboard-footprint:Diode_SOD123_2, F.Cu at (116.1, 208.2)
- added D24: D, SofleKeyboard-footprint:Diode_SOD123_2, F.Cu at (116.1, 210.8)
- added D25: D, SofleKeyboard-footprint:Diode_SOD123_2, F.Cu at (116.1, 213.3)
- added D26: D, SofleKeyboard-footprint:Diode_SOD123_2, F.Cu at (116.1, 215.8)
- added D27: D, SofleKeyboard-footprint:Diode_SOD123_2, F.Cu at (116.1, 218.4)
- added D28: D, SofleKeyboard-footprint:Diode_SOD123_2, F.Cu at (116.1, 220.9)
- added D29: D, SofleKeyboard-footprint:Diode_SOD123_2, F.Cu at (116.1, 223.5)
- added D3: D, SofleKeyboard-footprint:Diode_SOD123_2, F.Cu at (103.7, 210.8)
- added D30: D, SofleKeyboard-footprint:Diode_SOD123_2, F.Cu at (116.1, 226.1)
- added D31: D, SofleKeyboard-footprint:Diode_SOD123_2, F.Cu at (124.3, 205.7)
- added D32: D, SofleKeyboard-footprint:Diode_SOD123_2, F.Cu at (124.3, 208.2)
- added D33: D, SofleKeyboard-footprint:Diode_SOD123_2, F.Cu at (124.3, 210.8)
- added D34: D, SofleKeyboard-footprint:Diode_SOD123_2, F.Cu at (124.3, 213.3)
- added D35: D, SofleKeyboard-footprint:Diode_SOD123_2, F.Cu at (124.3, 215.8)
- added D36: D, SofleKeyboard-footprint:Diode_SOD123_2, F.Cu at (124.3, 218.4)
- added D37: D, SofleKeyboard-footprint:Diode_SOD123_2, F.Cu at (124.3, 220.9)
- added D38: D, SofleKeyboard-footprint:Diode_SOD123_2, F.Cu at (124.3, 223.5)
- added D39: D, SofleKeyboard-footprint:Diode_SOD123_2, F.Cu at (124.3, 226.1)
- added D4: D, SofleKeyboard-footprint:Diode_SOD123_2, F.Cu at (103.7, 213.3)
- added D40: D, SofleKeyboard-footprint:Diode_SOD123_2, F.Cu at (124.3, 228.6)
- added D41: D, SofleKeyboard-footprint:Diode_SOD123_2, F.Cu at (130.5, 205.7)
- added D42: D, SofleKeyboard-footprint:Diode_SOD123_2, F.Cu at (130.5, 208.2)
- added D43: D, SofleKeyboard-footprint:Diode_SOD123_2, F.Cu at (130.5, 210.8)
- added D44: D, SofleKeyboard-footprint:Diode_SOD123_2, F.Cu at (130.5, 213.3)
- added D45: D, SofleKeyboard-footprint:Diode_SOD123_2, F.Cu at (130.5, 215.8)
- added D46: D, SofleKeyboard-footprint:Diode_SOD123_2, F.Cu at (130.5, 218.4)
- added D47: D, SofleKeyboard-footprint:Diode_SOD123_2, F.Cu at (130.5, 220.9)
- added D48: D, SofleKeyboard-footprint:Diode_SOD123_2, F.Cu at (130.5, 223.5)
- added D49: D, SofleKeyboard-footprint:Diode_SOD123_2, F.Cu at (130.5, 226.1)
- added D50: D, SofleKeyboard-footprint:Diode_SOD123_2, F.Cu at (130.5, 228.6)
- added D51: D, SofleKeyboard-footprint:Diode_SOD123_2, F.Cu at (136.7, 205.7)
- added D52: D, SofleKeyboard-footprint:Diode_SOD123_2, F.Cu at (136.7, 208.2)
- added D53: D, SofleKeyboard-footprint:Diode_SOD123_2, F.Cu at (136.7, 210.8)
- added D54: D, SofleKeyboard-footprint:Diode_SOD123_2, F.Cu at (136.7, 213.3)
- added D55: D, SofleKeyboard-footprint:Diode_SOD123_2, F.Cu at (136.7, 215.8)
- added D56: D, SofleKeyboard-footprint:Diode_SOD123_2, F.Cu at (136.7, 218.4)
- added D57: D, SofleKeyboard-footprint:Diode_SOD123_2, F.Cu at (136.7, 220.9)
- added D58: D, SofleKeyboard-footprint:Diode_SOD123_2, F.Cu at (136.7, 223.5)
- added D59: D, SofleKeyboard-footprint:Diode_SOD123_2, F.Cu at (136.7, 226.1)
- added D6: D, SofleKeyboard-footprint:Diode_SOD123_2, F.Cu at (103.7, 215.8)
- added D60: D, SofleKeyboard-footprint:Diode_SOD123_2, F.Cu at (136.7, 228.6)
- added D61: D, SofleKeyboard-footprint:Diode_SOD123_2, F.Cu at (116.1, 228.6)
- added D7: D, SofleKeyboard-footprint:Diode_SOD123_2, F.Cu at (103.7, 218.4)
- added D8: D, SofleKeyboard-footprint:Diode_SOD123_2, F.Cu at (103.7, 220.9)
- added D9: D, SofleKeyboard-footprint:Diode_SOD123_2, F.Cu at (103.7, 223.5)
