File: Sofle_v2/PCB_TFTScreen/SofleKeyboard.kicad_sch (KiCad schematic)
At the start: 0 parts

Commit message: Update file
Other:
- sheet RGB Left renamed RGB Right
- sheet RGB Right: file RGB_Left.kicad_sch -> RGB_Right.kicad_sch
Changed lines of the file:
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@@
     (stroke (width 0.1524) (type solid))
     (fill (color 0 0 0 0.0000))
-    (property "Sheetname" "RGB Left" (at 50.8 56.4384 0)
+    (property "Sheetname" "RGB Right" (at 50.8 56.4384 0)
       (effects (font (size 1.27 1.27)) (justify left bottom))
     )
-    (property "Sheetfile" "RGB_Left.kicad_sch" (at 50.8 76.7846 0)
+    (property "Sheetfile" "RGB_Right.kicad_sch" (at 50.8 76.7846 0)
       (effects (font (size 1.27 1.27)) (justify left top))
     )
